File: HARDWARE/QuadSKPico.kicad_sch (KiCad schematic)
At the start: 131 parts, among them J1 BOOT, J2 AVR-JTAG-10, J8 ADDR, P1 USB_C_Plug_USB2.0, U1 TXS0108EPW, U10 RP2040, U11 PCM5122PW, U12 W25Q32RVXHJQ, U13 RP2040, U14 PCM5122PW, U15 W25Q32RVXHJQ, U2 PCM5122PW, U3 OPA2134, U4 MAX9723, U5 AP7365-33EG-13, U6 TXS0108EPW, U7 RP2040, U8 PCM5122PW, U9 W25Q32RVXHJQ, X1 DSC1001BI2-012.0000T

Commit message: Add files via upload
Parts:
- removed R?: 10k, Capacitor_SMD:C_0805_2012Metric_Pad1.18x1.45mm_HandSolder, symbol Device:R_Small_US
- added J5: MONO, Connector_PinHeader_2.54mm:PinHeader_1x02_P2.54mm_Vertical, symbol Connector_Generic:Conn_01x02
- added J6: HEADPHONE OUT, Connector_PinHeader_2.54mm:PinHeader_1x03_P2.54mm_Vertical, symbol Connector_Generic:Conn_01x03
- added J7: EVO64 SID2 Pin27, Connector_PinHeader_2.54mm:PinHeader_1x01_P2.54mm_Vertical, symbol Connector_Generic:Conn_01x01
- added R1: 4k7, Capacitor_SMD:C_0805_2012Metric_Pad1.18x1.45mm_HandSolder, symbol Device:R_Small_US
- R35, R37, R39: renamed from R?; value 10k -> 4k7
- U7: renamed from U3; footprint (none) -> Package_SO:SOIC-8_3.9x4.9mm_P1.27mm
- gave numbers to parts that had none: 7
- renumbered C10 to C1, C37 to C10, C34 to C11, C38 to C12, C32 to C13, C39 to C14, C40 to C15, C41 to C16, C42 to C17, C43 to C18, C44 to C19, C5 to C2, C30 to C20, C6 to C21, C29 to C22, C56 to C23, C46 to C24, C31 to C25, C11 to C26, C51 to C27, C57 to C28, C47 to C29, C28 to C3, C49 to C30, C48 to C31, C3 to C32, C19 to C33, C52 to C34, C58 to C35, C2 to C36, C25 to C37, C53 to C38, C59 to C39, C55 to C4, C50 to C40, C45 to C41, C14 to C42, C26 to C43, C54 to C44, C60 to C45, C7 to C46, C9 to C47, C27 to C48, C33 to C49, C1 to C5, C20 to C50, C21 to C51, C22 to C52, C23 to C53, C15 to C54, C16 to C55, C12 to C56, C13 to C57, C8 to C58, C17 to C59, C4 to C6, C18 to C60, C24 to C7, C35 to C8, C36 to C9, J8 to J2, J2 to J3, R19 to R10, R38 to R11, R22 to R12, R20 to R13, R24 to R14, R25 to R15, R26 to R16, R27 to R17, R28 to R18, R29 to R19, R14 to R2, R30 to R20, R31 to R21, R32 to R22, R36 to R23, R34 to R24, R33 to R25, R35 to R26, R11 to R27, R2 to R28, R10 to R29, R16 to R3, R5 to R30, R6 to R31, R1 to R32, R7 to R33, R12 to R36, R3 to R38, R15 to R4, R13 to R40, R4 to R41, R17 to R5, R37 to R6, R21 to R7, R18 to R8, R23 to R9, U5 to U1, U8 to U10, U14 to U12, U4 to U14, U1 to U15, U6 to U16, U9 to U18, U12 to U19, U15 to U20, U7 to U4, U10 to U5, U13 to U6, U2 to U9
Connections:
- net AUDOUT is gone; now on net OUTLP: S1.27 (AUDIO-OUT)
- net +3V3: now also R35.1, R37.1, R39.1, R1.1
- net +5V: no longer R35.1, R37.1, R39.1
- net BOOT: now also R1.2; no longer R30.1, R31.1, R32.1, R33.1
- net EP: now also C40.2, U10.11 (SDA/MOSI/ATT2), U10.12 (SCL/MC/ATT1), U10.13 (P0IO5/ATT0), U10.14 (P0IO4/MAST), U10.16 (ADR2/P0IO2/DOUT), U10.17 (MODE1), U10.18 (MODE2/MS), U11.11 (SDA/MOSI/ATT2), U11.12 (SCL/MC/ATT1), U11.13 (P0IO5/ATT0), U11.14 (P0IO4/MAST), U11.16 (ADR2/P0IO2/DOUT), U11.17 (MODE1), U11.18 (MODE2/MS), U12.11 (SDA/MOSI/ATT2), U12.12 (SCL/MC/ATT1), U12.13 (P0IO5/ATT0), U12.14 (P0IO4/MAST), U12.16 (ADR2/P0IO2/DOUT), U12.17 (MODE1), U12.18 (MODE2/MS), U9.11 (SDA/MOSI/ATT2), U9.12 (SCL/MC/ATT1), U9.13 (P0IO5/ATT0), U9.14 (P0IO4/MAST), U9.16 (ADR2/P0IO2/DOUT), U9.17 (MODE1), U9.18 (MODE2/MS), J6.1 (Pin_1)
- net OUTL: now also J6.2 (Pin_2)
- net OUTR: now also J6.3 (Pin_3)
- net OUTRP: now also J7.1 (Pin_1)
- net SUM_L: now reaches R12.1, R2.1, R3.1, R5.1, R7.2, R8.1, R9.1
- net SUM_L: now also J5.2 (Pin_2)
- net SUM_R: now reaches R14.1, R15.1, R16.1, R17.2, R18.1, R19.1, R21.1
- net SUM_R: now also J5.1 (Pin_1)
- new net BOOT0: R32.1
- new net BOOT1: R30.1
- new net BOOT2: R31.1
- new net BOOT3: R33.1
- no-connect marks 21 -> 22
Other:
- note added: "$D400"
- note added: "$D440"
- note added: "$D480"
- note added: "$D4C0"
- note added: "AUDIO"
- note added: "SID Socket"
- note added: "USB"
- moved on the sheet: C1, C10, C11, C12, C13, C14, C15, C16, C17, C18, C19, C2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

Commit message: Add files via upload
Parts:
- removed U15, U16: TXS0108EPW, Package_SO:TSSOP-20_4.4x6.5mm_P0.65mm, symbol Logic_LevelTranslator:TXS0108EPW
- added U15, U16: LSF0108BQ, Package_DFN_QFN:DHVQFN-20-1EP_2.5x4.5mm_P0.5mm_EP1x3mm, symbol CPU2:LSF0108BQ
Connections:
- net +3V3: now also U15.2 (VCCA), U16.2 (VCCA)
- net +5P: now also U15.19 (VCCB), U16.19 (VCCB)
- net A0: now also U16.18 (B1)
- net A1: now also U16.17 (B2)
- net A2: now also U16.16 (B3)
- net A3: now also U16.15 (B4)
- net A4: now also U16.14 (B5)
- net A5: now also U16.13 (B6)
- net A6: now also U16.12 (B7)
- net A7: now also U16.11 (B8)
- net D0: now also U15.18 (B1)
- net D1: now also U15.17 (B2)
- net D2: now also U15.16 (B3)
- net D3: now also U15.15 (B4)
- net D4: now also U15.14 (B5)
- net D5: now also U15.13 (B6)
- net D6: now also U15.12 (B7)
- net D7: now also U15.11 (B8)
- net ENTR: now also U15.20 (EN), U16.20 (EN)
- net EP: now also U15.1 (GND), U15.21 (MP), U16.1 (GND), U16.21 (MP)
- net LA0: now also U16.3 (A1)
- net LA1: now also U16.4 (A2)
- net LA2: now also U16.5 (A3)
- net LA3: now also U16.6 (A4)
- net LA4: now also U16.7 (A5)
- net LA5: now also U16.8 (A6)
- net LA6: now also U16.9 (A7)
- net LA7: now also U16.10 (A8)
- net LD0: now also U15.3 (A1)
- net LD1: now also U15.4 (A2)
- net LD2: now also U15.5 (A3)
- net LD3: now also U15.6 (A4)
- net LD4: now also U15.7 (A5)
- net LD5: now also U15.8 (A6)
- net LD6: now also U15.9 (A7)
- net LD7: now also U15.10 (A8)
Other:
- moved on the sheet: J4, J5, J6, J7
